Commit message: modified code to move robot base to be on the side wall

File: ur_description/urdf/ur5_robot.urdf.xacro (robot description, xacro)
@@ -6,11 +6,7 @@
   <!-- ur5 -->
   <xacro:include filename="$(find ur_description)/urdf/ur5.urdf.xacro" />
+  <!-- robot mount -->
+  <xacro:include filename="$(find ur_description)/urdf/hang_robot.xacro" />
   <!-- arm -->
   <xacro:ur5_robot prefix="" joint_limited="false"/>
-  <link name="world" />
-  <joint name="world_joint" type="fixed">
-    <parent link="world" />
-    <child link = "base_link" />
-    <origin xyz="0.0 0.0 0.0" rpy="0.0 0.0 0.0" />
-  </joint>
 </robot>
